Commit message: Commit message for changes in racecar_gazebo

File: racecar_description/urdf/macros.xacro (robot description, xacro)
@@ -4,5 +4,5 @@
 <xacro:macro name="chassis_inertial_params">
   <origin xyz="0.1477 0 0" rpy="0 0 0" />
-  <mass value="10.0" />
+  <mass value="4.0" />
   <inertia ixx="0.010609" ixy="0"          ixz="0"
                           iyy="0.050409"   iyz="0"
@@ -26,11 +26,4 @@
   <origin xyz="0 0 0" rpy="0 0 0" />
   <mass value="0.100" />
-  <inertia ixx="4E-06" ixy="0"           ixz="0"
-                            iyy="4E-06"  iyz="0"
-                                              izz="4E-06" />
-</xacro:macro>
-<xacro:macro name="hokuyo_inertial_params">
-  <origin xyz="0 0 0" rpy="0 0 0" />
-  <mass value="0.130" />
   <inertia ixx="4E-06" ixy="0"           ixz="0"
                             iyy="4E-06"  iyz="0"
@@ -97,8 +90,8 @@
     <type>transmission_interface/SimpleTransmission</type>
     <joint name="${name}_joint">
-      <hardwareInterface>hardware_interface/EffortJointInterface</hardwareInterface>
+      <hardwareInterface>EffortJointInterface</hardwareInterface>
     </joint>
     <actuator name="${name}_motor">
-      <hardwareInterface>hardware_interface/EffortJointInterface</hardwareInterface>
+      <hardwareInterface>EffortJointInterface</hardwareInterface>
       <mechanicalReduction>1</mechanicalReduction>
     </actuator>
@@ -109,8 +102,8 @@
     <type>transmission_interface/SimpleTransmission</type>
     <joint name="${name}_joint">
-      <hardwareInterface>hardware_interface/EffortJointInterface</hardwareInterface>
+      <hardwareInterface>EffortJointInterface</hardwareInterface>
     </joint>
     <actuator name="${name}_motor">
-      <hardwareInterface>hardware_interface/EffortJointInterface</hardwareInterface>
+      <hardwareInterface>EffortJointInterface</hardwareInterface>
       <mechanicalReduction>1</mechanicalReduction>
     </actuator>

File: racecar_description/urdf/racecar.xacro (robot description, xacro)
@@ -7,5 +7,5 @@
     <visual>
       <xacro:chassis_geometry/>
-      <material name="red" />
+      <material name="blue" />
     </visual>
   </link>
@@ -43,5 +43,5 @@
     <child link="left_rear_wheel" />
     <axis xyz="0 0 -1" />
-    <limit effort="10" velocity="1000" />
+    <limit effort="10" velocity="100" />
   </joint>
   <xacro:wheel_transmission name="left_rear_wheel" />
@@ -64,5 +64,5 @@
     <child link="right_rear_wheel" />
     <axis xyz="0 0 -1" />
-    <limit effort="10" velocity="1000" />
+    <limit effort="10" velocity="100" />
   </joint>
   <xacro:wheel_transmission name="right_rear_wheel" />
@@ -82,5 +82,5 @@
     <child link="left_steering_hinge" />
     <axis xyz="-1 0 0" />
-    <limit lower="-1.0" upper="1.0" effort="10" velocity="1000" />
+    <limit lower="-1.0" upper="1.0" effort="10" velocity="100" />
   </joint>
   <xacro:steering_hinge_transmission name="left_steering_hinge" />
@@ -100,5 +100,5 @@
     <child link="right_steering_hinge" />
     <axis xyz="-1 0 0" />
-    <limit lower="-1.0" upper="1.0" effort="10" velocity="1000" />
+    <limit lower="-1.0" upper="1.0" effort="10" velocity="100" />
   </joint>
   <xacro:steering_hinge_transmission name="right_steering_hinge" />
@@ -121,5 +121,5 @@
     <child link="left_front_wheel" />
     <axis xyz="0 0 -1" />
-    <limit effort="10" velocity="1000" />
+    <limit effort="10" velocity="100" />
   </joint>
   <xacro:wheel_transmission name="left_front_wheel" />
@@ -142,32 +142,34 @@
     <child link="right_front_wheel" />
     <axis xyz="0 0 -1" />
-    <limit effort="10" velocity="1000"/>
+    <limit effort="10" velocity="100"/>
   </joint>
   <xacro:wheel_transmission name="right_front_wheel" />
-  <!-- Add Hokuyo laser scanner -->
+  <joint name="rplidar_joint" type="fixed">
+    <axis xyz="0 1 0" />
+    <origin xyz="0.02 0 0.058" rpy="0 0 3.14"/>
+    <parent link="base_link"/>
+    <child link="laser"/>
+  </joint>
+  <!-- rplidar Laser -->
   <link name="laser">
-    <inertial>
-      <xacro:hokuyo_inertial_params />
-    </inertial>
-    <collision>
-      <origin xyz="0 0 0" rpy="0 0 0"/>
-      <geometry>
-        <box size="0.1 0.1 0.1"/>
-      </geometry>
-    </collision>
-    <visual>
-      <origin xyz="0 0 0" rpy="0 0 0"/>
-      <geometry>
-        <mesh filename="package://racecar_description/meshes/hokuyo.dae"/>
-        <material name="grey" />
-      </geometry>
-    </visual>
-  </link>
-  <joint name="hokuyo_joint" type="fixed">
-    <origin xyz="0.265 0.0 0.075" rpy="0 0 0"/>
-    <parent link="chassis" />
-    <child link="laser" />
-    <axis xyz="0 0 1" />
-  </joint>
+    <collision>
+      <origin xyz="0 0 0" rpy="1.5707 0 4.71"/>
+      <geometry>
+        <mesh filename="package://racecar_description/meshes/rplidar.stl" scale="0.001 0.001 0.001" />
+      </geometry>
+    </collision>
+    <visual>
+      <origin xyz="0 0 0" rpy="1.5707 0 4.71"/>
+      <geometry>
+        <mesh filename="package://racecar_description/meshes/rplidar.stl" scale="0.001 0.001 0.001" />
+      </geometry>
+      <material name="blue"/>
+    </visual>
+    <inertial>
+      <mass value="1e-5" />
+      <origin xyz="0 0 0" rpy="1.5707 0 4.71"/>
+      <inertia ixx="0" ixy="0" ixz="0" iyy="0" iyz="0" izz="0" />
+    </inertial>
+  </link>
   <!-- zed camera -->
   <link name="zed_camera_link">
@@ -192,5 +194,5 @@
   </link>
   <joint name="zed_camera_joint" type="fixed">
-    <origin xyz="0.390 0 0.2" rpy="0 0.2 0"/>
+    <origin xyz="0.390 0 0.04" rpy="0 0 0"/>
     <parent link="chassis"/>
     <child link="zed_camera_link"/>
